Commit message: going to use the action lib for square, the current ros controller does not work well in simulation

File: src/sevenbot_description/urdf/sevenbot.xacro (robot description, xacro)
@@ -3,4 +3,13 @@
   <xacro:include filename="$(find sevenbot_description)/urdf/sevenbot.gazebo" />
   <xacro:include filename="$(find sevenbot_description)/urdf/materials.xacro" />
+  <link name='dummy_link'>
+      <origin xyz="0.0 0 0.1" rpy=" 0 0 0"/>
+  </link>
+  <joint type="fixed" name="dummy_joint">
+    <origin xyz="0 0 0.1" rpy="0 0 0"/>
+    <child link="base_link"/>
+    <parent link="dummy_link"/>
+    <axis xyz="0 1 0" rpy="0 0 0"/>
+  </joint>
   <link name='base_link'>
     <pose>0 0 0.1 0 0 0</pose>
@@ -97,6 +106,6 @@
     <parent link="base_link"/>
     <axis xyz="0 1 0" rpy="0 0 0"/>
-    <limit effort="10000" velocity="1000"/>
-    <joint_properties damping="1.0" friction="1.0"/>
+    <limit effort="100" velocity="10"/>
+    <joint_properties damping="2.0" friction="1.5"/>
   </joint>
   <joint type="continuous" name="right_wheel_hinge">
@@ -105,6 +114,6 @@
     <parent link="base_link"/>
     <axis xyz="0 1 0" rpy="0 0 0"/>
-    <limit effort="10000" velocity="1000"/>
-    <joint_properties damping="1.0" friction="1.0"/>
+    <limit effort="100" velocity="10"/>
+    <joint_properties damping="1.0" friction="1.5"/>
   </joint>
 </robot>

Commit message: need to fix quaternion tmr

File: src/sevenbot_description/urdf/sevenbot.xacro (robot description, xacro)
@@ -4,16 +4,16 @@
   <xacro:include filename="$(find sevenbot_description)/urdf/materials.xacro" />
   <link name='dummy_link'>
-      <origin xyz="0.0 0 0.1" rpy=" 0 0 0"/>
+    <!-- <pose>0 0 0.1 0 0 0</pose> -->
+    <origin xyz="0.0 0 0.1" rpy=" 0 0 0"/>
   </link>
   <joint type="fixed" name="dummy_joint">
     <origin xyz="0 0 0.1" rpy="0 0 0"/>
+    <parent link="dummy_link"/>
     <child link="base_link"/>
-    <parent link="dummy_link"/>
-    <axis xyz="0 1 0" rpy="0 0 0"/>
+    <axis xyz="0 0 1" rpy="0 0 0"/>
   </joint>
   <link name='base_link'>
-    <pose>0 0 0.1 0 0 0</pose>
     <inertial>
-      <mass value="15.0"/>
+      <mass value="5.0"/>
       <origin xyz="0.0 0 0.1" rpy=" 0 0 0"/>
       <inertia
